File: CAD/Comms.kicad_sch (KiCad schematic)
At the start: 87 parts, among them J27 uSD_Socket, J32 Conn_01x02, J43 USB, J46 ETHERNET, J9 Conn_01x02, Q1 BC807, U13 MCP2542, U15 MCP2542, U16 KSZ8081RNACA, U17 74LVC2G125, U19 74LVC2G34, U3 EMIF06, U5 RClamp0504FB, U7 AP22816AKEWT, X2 25Mhz

Commit message: Misc Cleanup
Changed lines of the file:
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@@
 		(dnp no)
 		(property "Reference" "R122"
-			(at 60.325 227.33 90)
+			(at 59.69 222.25 90)
 			(effects
 				(font
@@
 		)
 		(property "Value" "27K"
-			(at 57.785 222.25 90)
+			(at 59.69 227.33 90)
 			(effects
 				(font

Commit message: Part Alternatives
Changed some alternatives for certain parts as they are out of stock and some won't come in until March 27
Also changed C6 so it uses the same cap as C29 so that manufacturing costs are lower
Parts:
- R11, R12, R122, R13, R81: Part Number AC0402FR-0727KL -> AC0402FR-0727KL or AF0402FR-0727KL
- U17: Part Number 74LVC2G125HD4-7 -> 74LVC2G125HD4-7 or 74LVC2G125GT,115
Changed lines of the file:
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@@
 			)
 		)
-		(property "Part Number" "AC0402FR-0727KL"
+		(property "Part Number" "AC0402FR-0727KL or AF0402FR-0727KL"
 			(at 59.69 224.79 0)
 			(hide yes)
@@
 			)
 		)
-		(property "Part Number" "AC0402FR-0727KL"
+		(property "Part Number" "AC0402FR-0727KL or AF0402FR-0727KL"
 			(at 266.7 205.74 0)
 			(hide yes)
@@
 			)
 		)
-		(property "Part Number" "AC0402FR-0727KL"
+		(property "Part Number" "AC0402FR-0727KL or AF0402FR-0727KL"
 			(at 181.61 204.47 0)
 			(hide yes)
@@
 			)
 		)
-		(property "Part Number" "AC0402FR-0727KL"
+		(property "Part Number" "AC0402FR-0727KL or AF0402FR-0727KL"
 			(at 175.26 204.47 0)
 			(hide yes)
@@
 			)
 		)
-		(property "Part Number" "AC0402FR-0727KL"
+		(property "Part Number" "AC0402FR-0727KL or AF0402FR-0727KL"
 			(at 261.62 215.9 0)
 			(hide yes)
@@
 			)
 		)
-		(property "Part Number" "74LVC2G125HD4-7"
+		(property "Part Number" "74LVC2G125HD4-7 or 74LVC2G125GT,115"
 			(at 201.93 194.945 0)
 			(hide yes)

Commit message: Added support for KiPIDA
New analysis tool that allows for thermal analysis.
Currently only DC Simulation and 3D Thermal Simulation is setup.
Connections:
- net 5V_INT renamed +5V_INT
Changed lines of the file:
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@@
 		)
 	)
-	(global_label "5V_INT"
+	(global_label "+5V_INT"
 		(shape input)
 		(at 40.64 322.58 180)
@@
 		)
 	)
-	(global_label "5V_INT"
+	(global_label "+5V_INT"
 		(shape input)
 		(at 52.07 26.67 90)
@@
 		)
 	)
-	(global_label "5V_INT"
+	(global_label "+5V_INT"
 		(shape input)
 		(at 49.53 91.44 180)
