File: CAD/Htr_Fan.kicad_sch (KiCad schematic)
At the start: 49 parts, among them J29 V_OUT_6-9 Select, J52 V_OUT_3-5 Select, Q25 Q_DUAL_NMOS, Q26 Q_DUAL_NMOS, Q27 Q_DUAL_NMOS, U12 74HCT2G34GW,125, U8 74HCT365, U9 74HCT365

Commit message: Added support for KiPIDA
New analysis tool that allows for thermal analysis.
Currently only DC Simulation and 3D Thermal Simulation is setup.
Changed lines of the file:
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@@
 		)
 	)
-	(global_label "5V_INT"
+	(global_label "+5V_INT"
 		(shape input)
 		(at 76.2 215.9 180)
@@
 		)
 	)
-	(global_label "5V_INT"
+	(global_label "+5V_INT"
 		(shape input)
 		(at 191.77 215.9 180)
@@
 		)
 	)
-	(global_label "5V_INT"
+	(global_label "+5V_INT"
 		(shape input)
 		(at 175.26 154.94 180)
