File: CAD/Stepper_Drv.kicad_sch (KiCad schematic)
At the start: 28 parts, among them U1 SN74F125DR, U14 SN74LVC4245APWR, U2 SN74F125DR, U21 SN74F125DR, U22 SN74F125DR, U25 SN74LVC4245APWR, U26 SN74LVC4245APWR, U6 SN74F125DR

Commit message: Added support for KiPIDA
New analysis tool that allows for thermal analysis.
Currently only DC Simulation and 3D Thermal Simulation is setup.
Connections:
- net 5V_INT renamed +5V_INT
Changed lines of the file:
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@@
 		)
 	)
-	(global_label "5V_INT"
+	(global_label "+5V_INT"
 		(shape input)
 		(at 246.38 217.17 180)
@@
 		)
 	)
-	(global_label "5V_INT"
+	(global_label "+5V_INT"
 		(shape input)
 		(at 198.12 53.34 90)
@@
 		)
 	)
-	(global_label "5V_INT"
+	(global_label "+5V_INT"
 		(shape input)
 		(at 62.23 154.94 180)
@@
 		)
 	)
-	(global_label "5V_INT"
+	(global_label "+5V_INT"
 		(shape input)
 		(at 153.67 214.63 180)
@@
 		)
 	)
-	(global_label "5V_INT"
+	(global_label "+5V_INT"
 		(shape input)
 		(at 196.85 154.94 180)
@@
 		)
 	)
-	(global_label "5V_INT"
+	(global_label "+5V_INT"
 		(shape input)
 		(at 123.19 50.8 90)
@@
 		)
 	)
-	(global_label "5V_INT"
+	(global_label "+5V_INT"
 		(shape input)
 		(at 33.02 50.8 90)
@@
 		)
 	)
-	(global_label "5V_INT"
+	(global_label "+5V_INT"
 		(shape input)
 		(at 71.12 215.9 180)
