File: CAD/Headers.kicad_sch (KiCad schematic)
At the start: 59 parts, among them J1 SWD, J10 OUT_0, J11 OUT_1, J12 OUT_2, J13 TEMP_0, J14 TEMP_1, J15 TEMP_2, J16 EXPANSION, J17 ESP_DB, J18 250-502/000-006, J19 A2543WV-5P, J2 A2543WV-2P, J20 IO_1, J21 IO_2, J22 A2543WV-2P, J23 CAN_1_OUT, J24 DRIVER_2, J25 DRIVER_1, J26 DRIVER_0, J28 SPI_DB, J3 OUT_6, J31 IO_3, J33 A2543WV-4P, J34 A2543WV-4P, J35 DRIVER_3, J36 DRIVER_4, J37 DRIVER_5, J38 CAN_0_OUT, J39 PANELDUE_SD, J4 OUT_7, J41 TEMP_3, J42 DS_LED, J44 IO_7_ISO_OUT, J47 IO_8_ISO_OUT, J48 SBC, J5 OUT_8, J50 EXT_5V_IN, J51 IO_4, J53 IO_5, J54 IO_6, J55 IO_7, J56 IO_8, J59 A2543WV-2P, J6 OUT_3, J60 A2543WV-2P, J61 IO_7_ISO_IN, J62 IO_8_ISO_IN, J7 OUT_4, J8 OUT_5

Commit message: Change P41 on J16
P41-NC changed -> P41-Erase
Connections:
- net ERASE: now reaches J16.41
- no-connect marks 26 -> 25
Changed lines of the file:
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@@
 	)
 	(no_connect
-		(at 105.41 340.36)
-	)
-	(no_connect
 		(at 105.41 294.64)
 	)
@@
 			(effects
 				(font
+					(size 1.27 1.27)
+				)
+				(justify right)
+				(hide yes)
+			)
+		)
+	)
+	(global_label "ERASE"
+		(shape input)
+		(at 105.41 340.36 180)
+		(fields_autoplaced yes)
+		(effects
+			(font
+				(size 1.27 1.27)
+			)
+			(justify right)
+		)
+		(property "Intersheetrefs" "${INTERSHEET_REFS}"
+			(at 97.2129 340.36 0)
+			(effects
+				(font

Commit message: Add F8 to fabrication files and SBC optional
Added fuse to fuse holder and SBC connector is now DnP by default, it can be soldered on if neeeded
Parts:
- J48: now not fitted; now left out of the parts list
Changed lines of the file:
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@@
 		(unit 1)
 		(exclude_from_sim no)
-		(in_bom yes)
+		(in_bom no)
 		(on_board yes)
-		(dnp no)
+		(dnp yes)
 		(property "Reference" "J48"
 			(at 202.565 81.28 0)

Commit message: 12V Converter Done
New 12V Converter, outputs to J22
Parts:
- J22: footprint Connector_Molex:Wurth_61900211121-1x02_P2.54mm_Vertical-(Molex_KK-254_AE-6410-02Acompatible) -> Connector_JST:JST_XH_B2B-XH-A_1x02_P2.50mm_Vertical; LCSC C239362 -> C158012; Part Number A2543WV-2P -> B2B-XH-A(LF)(SN); now fitted; now in the parts list
Connections:
- net 12V_EXT renamed 12V_BUCK_OUT
Other:
- note removed: "additional 12V supply if a VFD convertor is used"
Changed lines of the file:
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@@
 		)
 	)
-	(text "additional 12V supply if\na VFD convertor is used"
-		(exclude_from_sim no)
-		(at 48.26 160.401 0)
-		(effects
-			(font
-				(size 0.7112 0.7112)
-			)
-			(justify left bottom)
-		)
-	)
 	(text "SWD"
 		(exclude_from_sim no)
@@
 	(wire
 		(pts
-			(xy 36.83 160.655) (xy 36.83 163.83)
-		)
-		(stroke
-			(width 0)
-			(type default)
-		)
-	)
-	(wire
-		(pts
 			(xy 102.235 104.775) (xy 105.41 104.775)
 		)
@@
 	(wire
 		(pts
-			(xy 39.37 160.655) (xy 36.83 160.655)
-		)
-		(stroke
-			(width 0)
-			(type default)
-		)
-	)
-	(wire
-		(pts
 			(xy 193.675 104.14) (xy 196.85 104.14)
 		)
@@
 	(wire
 		(pts
-			(xy 106.045 99.695) (xy 101.6 99.695)
+			(xy 17.78 158.75) (xy 39.37 158.75)
 		)
 		(stroke
@@
 	(wire
 		(pts
-			(xy 141.605 107.95) (xy 144.145 107.95)
+			(xy 106.045 99.695) (xy 101.6 99.695)
 		)
 		(stroke
@@
 	(wire
 		(pts
-			(xy 233.045 120.015) (xy 211.455 120.015)
+			(xy 141.605 107.95) (xy 144.145 107.95)
 		)
 		(stroke
@@
 	(wire
 		(pts
-			(xy 106.045 138.43) (xy 101.6 138.43)
+			(xy 233.045 120.015) (xy 211.455 120.015)
 		)
 		(stroke
@@
 	(wire
 		(pts
-			(xy 138.43 270.51) (xy 160.02 270.51)
+			(xy 106.045 138.43) (xy 101.6 138.43)
 		)
 		(stroke
@@
 	(wire
 		(pts
-			(xy 105.41 144.78) (xy 105.41 146.685)
+			(xy 138.43 270.51) (xy 160.02 270.51)
 		)
 		(stroke
@@
 	(wire
 		(pts
-			(xy 134.62 138.43) (xy 134.62 153.67)
+			(xy 105.41 144.78) (xy 105.41 146.685)
 		)
 		(stroke
@@
 	(wire
 		(pts
-			(xy 35.56 26.67) (xy 35.56 25.4)
+			(xy 134.62 138.43) (xy 134.62 153.67)
 		)
 		(stroke
@@
 	(wire
 		(pts
-			(xy 33.655 158.115) (xy 39.37 158.115)
+			(xy 35.56 26.67) (xy 35.56 25.4)
 		)
 		(stroke
@@
 	(wire
 		(pts
+			(xy 17.78 162.56) (xy 17.78 158.75)
+		)
+		(stroke
+			(width 0)
+			(type default)
+		)
+	)
+	(wire
+		(pts
 			(xy 106.045 133.35) (xy 101.6 133.35)
 		)
@@
 		)
 	)
-	(global_label "12V_EXT"
-		(shape input)
-		(at 33.655 158.115 180)
-		(fields_autoplaced yes)
-		(effects
-			(font
-				(size 1.1938 1.1938)
-			)
-			(justify right)
-		)
-		(property "Intersheetrefs" "${INTERSHEET_REFS}"
-			(at 24.1305 158.115 0)
-			(effects
-				(font
-					(size 1.27 1.27)
-				)
-				(justify right)
-				(hide yes)
-			)
-		)
-	)
 	(global_label "IO_5_OUT_ISO_POS"
 		(shape output)
@@
 		)
 	)
+	(global_label "12V_BUCK_OUT"
+		(shape input)
+		(at 39.37 161.29 180)
+		(fields_autoplaced yes)
+		(effects
+			(font
+				(size 1.524 1.524)
+			)
+			(justify right)
+		)
+		(property "Intersheetrefs" "${INTERSHEET_REFS}"
+			(at 19.519 161.29 0)
+			(effects
+				(font
+					(size 1.27 1.27)
+				)
+				(justify right)
+				(hide yes)
+			)
+		)
+	)
 	(global_label "V_OUT_LC_2"
 		(shape input)
@@
 	)
 	(symbol
-		(lib_id "Connector_Generic:Conn_01x02")
-		(at 44.45 158.115 0)
-		(unit 1)
-		(exclude_from_sim no)
-		(in_bom no)
-		(on_board no)
-		(dnp yes)
-		(property "Reference" "J22"
-			(at 44.45 155.575 0)
-			(effects
-				(font
-					(size 1.016 1.016)
-				)
-			)
-		)
-		(property "Value" "A2543WV-2P"
-			(at 46.99 159.131 90)
-			(effects
-				(font
-					(size 1.016 1.016)
-				)
-				(hide yes)
-			)
-		)
-		(property "Footprint" "Connector_Molex:Wurth_61900211121-1x02_P2.54mm_Vertical-(Molex_KK-254_AE-6410-02Acompatible)"
-			(at 44.45 158.115 0)
-			(effects
-				(font
-					(size 1.524 1.524)
-				)
-				(hide yes)
-			)
-		)
-		(property "Datasheet" ""
-			(at 44.45 158.115 0)
-			(effects
-				(font
-					(size 1.524 1.524)
-				)
-				(hide yes)
-			)
-		)
-		(property "Description" "12V+ GND"
-			(at 46.99 159.385 90)
-			(effects
-				(font
-					(size 1.27 1.27)
-				)
-			)
-		)
-		(property "Part Number" "A2543WV-2P"
-			(at 44.45 158.115 0)
-			(effects
-				(font
-					(size 1.27 1.27)
-				)
-				(hide yes)
-			)
-		)
-		(property "LCSC" "C239362"
-			(at 44.45 158.115 0)
-			(effects
-				(font
-					(size 1.524 1.524)
-				)
-				(hide yes)
-			)
-		)
-		(property "RotOffset" "180"
-			(at 44.45 158.115 0)
-			(effects
-				(font
-					(size 1.524 1.524)
-				)
-				(hide yes)
-			)
-		)
-		(pin "1"
-		)
-		(pin "2"
-		)
-		(instances
-			(project ""
-				(path "/94813053-1316-4754-9fb4-4dbbf7dc780d/00000000-0000-0000-0000-000050656780"
-					(reference "J22")
-					(unit 1)
-				)
-			)
-		)
-	)
-	(symbol
 		(lib_name "GND_2")
 		(lib_id "Duet3:GND")
-		(at 36.83 163.83 0)
+		(at 17.78 162.56 0)
 		(unit 1)
 		(exclude_from_sim no)
@@
 		(dnp no)
 		(property "Reference" "#PWR0147"
-			(at 36.83 163.83 0)
+			(at 17.78 162.56 0)
 			(effects
 				(font
@@
 		)
 		(property "Value" "GND"
-			(at 36.83 165.608 0)
+			(at 17.78 164.338 0)
 			(effects
 				(font
@@
 		)
 		(property "Footprint" ""
-			(at 36.83 163.83 0)
+			(at 17.78 162.56 0)
 			(effects
 				(font
@@
 		)
 		(property "Datasheet" ""
-			(at 36.83 163.83 0)
+			(at 17.78 162.56 0)
 			(effects
 				(font
@@
 		)
 		(property "Description" ""
-			(at 36.83 163.83 0)
+			(at 17.78 162.56 0)
 			(effects
 				(font
@@
 					(unit 1)
 				)
+			)
+		)
+	)
+	(symbol
+		(lib_id "Connector_Generic:Conn_01x02")
+		(at 44.45 161.29 0)
+		(mirror x)
+		(unit 1)
+		(exclude_from_sim no)
+		(in_bom yes)
+		(on_board yes)
+		(dnp no)
+		(property "Reference" "J22"
+			(at 44.45 156.21 0)
+			(effects
+				(font
+					(size 1.016 1.016)
+				)
+			)
+		)
+		(property "Value" "A2543WV-2P"
+			(at 46.99 160.02 90)
+			(effects
+				(font
+					(size 1.016 1.016)
+				)
+				(hide yes)
+			)
+		)
+		(property "Footprint" "Connector_JST:JST_XH_B2B-XH-A_1x02_P2.50mm_Vertical"
+			(at 44.45 161.29 0)
+			(effects
+				(font
+					(size 1.524 1.524)
+				)
+				(hide yes)
+			)
+		)
+		(property "Datasheet" ""
+			(at 44.45 161.29 0)
+			(effects
+				(font
+					(size 1.524 1.524)
+				)
+				(hide yes)
+			)
+		)
+		(property "Description" "12V OUT"
+			(at 47.498 159.766 90)
+			(effects
+				(font
+					(size 1.27 1.27)
+				)
+			)
+		)
+		(property "Part Number" "B2B-XH-A(LF)(SN)"
+			(at 44.45 161.29 0)
+			(effects
+				(font
+					(size 1.27 1.27)
+				)
+				(hide yes)
+			)
+		)
+		(property "LCSC" "C158012"
+			(at 44.45 161.29 0)
+			(effects
+				(font
+					(size 1.524 1.524)
+				)
+				(hide yes)
+			)
+		)
+		(property "RotOffset" "180"
+			(at 44.45 161.29 0)
+			(effects
+				(font
+					(size 1.524 1.524)
+				)
+				(hide yes)
+			)
+		)
+		(pin "1"
+		)
+		(pin "2"
+		)
+		(instances
+			(project "Duet3_MB_3DP"
+				(path "/94813053-1316-4754-9fb4-4dbbf7dc780d/00000000-0000-0000-0000-000050656780"
+					(reference "J22")
+					(unit 1)
+				)

Commit message: Add Wattage Info
Other:
- note added: "Always on FAN for board cooling MAX 1 AMP. DO NOT EXCEED"
- note removed: "Always on FAN for board cooling"
Changed lines of the file:
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@@
 		)
 	)
-	(text "Always on FAN for board cooling"
+	(text "Always on FAN for board cooling\nMAX 1 AMP. DO NOT EXCEED"
 		(exclude_from_sim no)
 		(at 46.355 81.026 0)

Commit message: Added support for KiPIDA
New analysis tool that allows for thermal analysis.
Currently only DC Simulation and 3D Thermal Simulation is setup.
Connections:
- net 12V_BUCK_OUT renamed +12V_BUCK_OUT
- net 5V_EXT renamed +5V_EXT
- net 5V_EXT_INPUT renamed +5V_EXT_INPUT
- net 5V_SBC renamed +5V_SBC
Changed lines of the file:
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@@
 		)
 	)
-	(global_label "5V_EXT"
+	(global_label "+5V_EXT"
 		(shape input)
 		(at 101.6 164.465 180)
@@
 		)
 	)
-	(global_label "5V_EXT_INPUT"
+	(global_label "+5V_EXT_INPUT"
 		(shape input)
 		(at 32.385 44.45 180)
@@
 		)
 	)
-	(global_label "5V_EXT"
+	(global_label "+5V_EXT"
 		(shape input)
 		(at 101.6 128.27 180)
@@
 		)
 	)
-	(global_label "5V_EXT"
+	(global_label "+5V_EXT"
 		(shape input)
 		(at 105.41 187.96 180)
@@
 		)
 	)
-	(global_label "5V_SBC"
+	(global_label "+5V_SBC"
 		(shape input)
 		(at 214.63 47.625 0)
@@
 		)
 	)
-	(global_label "5V_EXT"
+	(global_label "+5V_EXT"
 		(shape input)
 		(at 141.605 97.79 180)
@@
 		)
 	)
-	(global_label "5V_EXT"
+	(global_label "+5V_EXT"
 		(shape input)
 		(at 101.6 92.075 180)
@@
 		)
 	)
-	(global_label "5V_EXT"
+	(global_label "+5V_EXT"
 		(shape input)
 		(at 198.12 20.955 180)
@@
 		)
 	)
-	(global_label "5V_EXT"
+	(global_label "+5V_EXT"
 		(shape input)
 		(at 138.43 137.16 90)
@@
 		)
 	)
-	(global_label "5V_EXT"
+	(global_label "+5V_EXT"
 		(shape input)
 		(at 101.6 109.855 180)
@@
 		)
 	)
-	(global_label "12V_BUCK_OUT"
+	(global_label "+12V_BUCK_OUT"
 		(shape input)
 		(at 39.37 161.29 180)
@@
 		)
 	)
-	(global_label "5V_EXT"
+	(global_label "+5V_EXT"
 		(shape input)
 		(at 101.6 73.66 180)
@@
 		)
 	)
-	(global_label "5V_EXT"
+	(global_label "+5V_EXT"
 		(shape input)
 		(at 101.6 146.685 180)

Commit message: Misc Changes to 12V
Changed inductor on 12V Buck to fit within amperage limits.
Also removed a test point as it is not needed.
Parts:
- removed TP39: VREFP, 3DPotter:TestPoint_Pad_D1.5mm, symbol Duet3:TP
Changed lines of the file:
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@@
 		)
 	)
-	(global_label "VREFP"
-		(shape input)
-		(at 258.445 24.765 180)
-		(fields_autoplaced yes)
-		(effects
-			(font
-				(size 1.1938 1.1938)
-			)
-			(justify right)
-		)
-		(property "Intersheetrefs" "${INTERSHEET_REFS}"
-			(at -33.655 -41.91 0)
-			(hide yes)
-			(show_name no)
-			(do_not_autoplace no)
-			(effects
-				(font
-					(size 1.27 1.27)
-				)
-			)
-		)
-	)
 	(global_label "D_5_STEP_NEG"
 		(shape input)
@@
 					(unit 1)
 				)
-			)
-		)
-	)
-	(symbol
-		(lib_id "Duet3:TP")
-		(at 258.445 24.765 270)
-		(unit 1)
-		(body_style 1)
-		(exclude_from_sim no)
-		(in_bom no)
-		(on_board yes)
-		(in_pos_files yes)
-		(dnp no)
-		(property "Reference" "TP39"
-			(at 268.605 24.765 90)
-			(show_name no)
-			(do_not_autoplace no)
-			(effects
-				(font
-					(size 1.524 1.524)
-				)
-			)
-		)
-		(property "Value" "VREFP"
-			(at 267.335 24.765 0)
-			(hide yes)
-			(show_name no)
-			(do_not_autoplace no)
-			(effects
-				(font
-					(size 1.524 1.524)
-				)
-			)
-		)
-		(property "Footprint" "3DPotter:TestPoint_Pad_D1.5mm"
-			(at 258.445 24.765 0)
-			(hide yes)
-			(show_name no)
-			(do_not_autoplace no)
-			(effects
-				(font
-					(size 1.524 1.524)
-				)
-			)
-		)
-		(property "Datasheet" ""
-			(at 258.445 24.765 0)
-			(hide yes)
-			(show_name no)
-			(do_not_autoplace no)
-			(effects
-				(font
-					(size 1.524 1.524)
-				)
-			)
-		)
-		(property "Description" ""
-			(at 258.445 24.765 0)
-			(hide yes)
-			(show_name no)
-			(do_not_autoplace no)
-			(effects
-				(font
-					(size 1.27 1.27)
-				)
-			)
-		)
-		(property "Part Number" "Virtual Component DNP"
-			(at 258.445 24.765 0)
-			(hide yes)
-			(show_name no)
-			(do_not_autoplace no)
-			(effects
-				(font
-					(size 1.27 1.27)
-				)
-			)
-		)
-		(pin "1"
-		)
-		(instances
-			(project "Duet3_MB_3DP"
-				(path "/94813053-1316-4754-9fb4-4dbbf7dc780d/00000000-0000-0000-0000-000050656780"
-					(reference "TP39")
-					(unit 1)
-				)
